Commit message: stable version for lidar and imu

File: urdf/test2.urdf (robot description, URDF)
Before this commit: robot cartographer_my_robot, 5 links, 4 joints
Joints:
- joint gps_joint: origin xyz=0.6 0. 0.15 rpy=0.0 0.0 0.0 -> xyz=1.02 0. 0.15 rpy=0.0 0.0 0.0

Commit message: fix bug in accumulating cloud

File: urdf/test2.urdf (robot description, URDF)
Before this commit: robot cartographer_my_robot, 5 links, 4 joints
Joints:
- joint gps_joint: origin xyz=1.02 0. 0.15 rpy=0.0 0.0 0.0 -> xyz=0.05 0.35 -0.1 rpy=0.0 0.0 0.0
- joint imu_link_joint: origin xyz=0 0.0 0.0 rpy=0.0 0.0 3.1415927 -> xyz=0 0.0 0.0 rpy=0.0 0.0 0.0
- joint velodyne_joint: origin xyz=-0.04 0.02 +0.30 rpy=0.0 0.0 3.1415927 -> xyz=0.04 -0.02 +0.30 rpy=0.0 0.0 0.0
